Commit message: rotating oxbstacles

File: aerialist/resources/simulation/box.xacro (robot description, xacro)
@@ -11,4 +11,5 @@
         <box size="$(arg l) $(arg w) $(arg h)"/>
       </geometry>
+      <origin xyz="${$(arg l)/2} ${$(arg w)/2} ${$(arg h)/2}"/>
     </collision>
     <visual>
@@ -16,4 +17,5 @@
         <box size="$(arg l) $(arg w) $(arg h)"/>
       </geometry>
+      <origin xyz="${$(arg l)/2} ${$(arg w)/2} ${$(arg h)/2}"/>
     </visual>
     <inertial>

Commit message: fix rotation difference in gazebo and obstacle center position

File: aerialist/resources/simulation/box.xacro (robot description, xacro)
@@ -11,5 +11,5 @@
         <box size="$(arg l) $(arg w) $(arg h)"/>
       </geometry>
-      <origin xyz="${$(arg l)/2} ${$(arg w)/2} ${$(arg h)/2}"/>
+      <!-- <origin xyz="${-$(arg l)/2} ${-$(arg w)/2} ${$(arg h)/2}"/> -->
     </collision>
     <visual>
@@ -17,5 +17,5 @@
         <box size="$(arg l) $(arg w) $(arg h)"/>
       </geometry>
-      <origin xyz="${$(arg l)/2} ${$(arg w)/2} ${$(arg h)/2}"/>
+      <!-- <origin xyz="${-$(arg l)/2} ${-$(arg w)/2} ${$(arg h)/2}"/> -->
     </visual>
     <inertial>

Commit message: Changes for entering pattern in Aerialist via launch file

File: aerialist/resources/simulation/box.xacro (robot description, xacro)
@@ -5,6 +5,9 @@
   <xacro:arg name="w" default = "1"/>
   <xacro:arg name="h" default = "1" />
+  <xacro:arg name="pattern" default=""/>
+  <xacro:property name="path" value="/home/prasun/Aerialist/aerialist/resources/simulation/models/big_box/meshes/big_box_"/>
+  <xacro:property name="extension" value=".dae"/>
   <link name="$(arg name)">
-    <static>true</static>
+    <static>false</static>
     <collision>
       <geometry>
@@ -15,5 +18,6 @@
     <visual>
       <geometry>
-        <box size="$(arg l) $(arg w) $(arg h)"/>
+        <!--<box size="$(arg l) $(arg w) $(arg h)"/>-->
+        <mesh filename = "${path}$(arg pattern)${extension}" scale="1.0 1.0 1.0"/>
       </geometry>
       <!-- <origin xyz="${-$(arg l)/2} ${-$(arg w)/2} ${$(arg h)/2}"/> -->

Commit message: Changes for downloading the intermediate images

File: aerialist/resources/simulation/box.xacro (robot description, xacro)
@@ -5,4 +5,8 @@
   <xacro:arg name="w" default = "1"/>
   <xacro:arg name="h" default = "1" />
+  <xacro:arg name="pattern" default=""/>
+  <!-- <xacro:property name="path" value="/home/prasun/Aerialist/aerialist/resources/simulation/models/big_box/meshes/big_box_"/> -->
+ <xacro:property name="path" value="/src/aerialist/aerialist/resources/simulation/models/big_box/meshes/big_box_"/>
+  <xacro:property name="extension" value=".dae"/>
   <link name="$(arg name)">
     <static>true</static>
@@ -15,11 +19,12 @@
     <visual>
       <geometry>
-        <box size="$(arg l) $(arg w) $(arg h)"/>
+        <mesh filename = "${path}$(arg pattern)${extension}" scale="6.0 6.0 10.0"/>
+        <!-- <box size="$(arg l) $(arg w) $(arg h)"/> -->
       </geometry>
       <!-- <origin xyz="${-$(arg l)/2} ${-$(arg w)/2} ${$(arg h)/2}"/> -->
     </visual>
     <inertial>
-      <mass value="1"/>
-      <inertia ixx="1.0" ixy="0.0" ixz="0.0" iyy="1.0" iyz="0.0" izz="1.0"/>
+      <mass value="100"/>
+      <inertia ixx="1088.0" ixy="0.0" ixz="0.0" iyy="550.0" iyz="0.0" izz="1088.0"/>
     </inertial>
   </link>

Commit message: Refactoring and organizing code

File: aerialist/resources/simulation/box.xacro (robot description, xacro)
@@ -6,6 +6,7 @@
   <xacro:arg name="h" default = "1" />
   <xacro:arg name="pattern" default=""/>
-  <!-- <xacro:property name="path" value="/home/prasun/Aerialist/aerialist/resources/simulation/models/big_box/meshes/big_box_"/> -->
- <xacro:property name="path" value="/src/aerialist/aerialist/resources/simulation/models/big_box/meshes/big_box_"/>
+  <!-- <xacro:arg name="path1" default=""> -->
+  <xacro:arg name="path" default=""/>
+ <!-- <xacro:property name="path" value="/src/aerialist/aerialist/resources/simulation/models/big_box/meshes/big_box_"/> -->
   <xacro:property name="extension" value=".dae"/>
   <link name="$(arg name)">
@@ -19,5 +20,5 @@
     <visual>
       <geometry>
-        <mesh filename = "${path}$(arg pattern)${extension}" scale="6.0 6.0 10.0"/>
+        <mesh filename = "$(arg path)$(arg pattern)${extension}" scale="6.0 6.0 10.0"/>
         <!-- <box size="$(arg l) $(arg w) $(arg h)"/> -->
       </geometry>

Commit message: handle 3rd and 4th obstacle in Docker Agent + stable obstacles

File: aerialist/resources/simulation/box.xacro (robot description, xacro)
@@ -5,4 +5,7 @@
   <xacro:arg name="w" default = "1"/>
   <xacro:arg name="h" default = "1" />
+  <xacro:arg name="mass" default="1000" />
+  <!-- <xacro:property name="volume" value="$(arg l) * $(arg w) * $(arg h)" />
+  <xacro:property name="mass" value="$(arg density) * ${volume}" /> -->
   <link name="$(arg name)">
     <static>true</static>
@@ -20,6 +23,6 @@
     </visual>
     <inertial>
-      <mass value="1"/>
-      <inertia ixx="1.0" ixy="0.0" ixz="0.0" iyy="1.0" iyz="0.0" izz="1.0"/>
+      <mass value="$(arg mass)"/>
+      <inertia ixx="${0.083*$(arg mass)*($(arg w)*$(arg w)+$(arg h)*$(arg h))}" ixy="0" ixz="0" iyy="${0.083*$(arg mass)*($(arg l)*$(arg l)+$(arg h)*$(arg h))}" iyz="0" izz="${0.083*$(arg mass)*($(arg l)*$(arg l)+$(arg w)*$(arg w))}"/>
     </inertial>
   </link>

Commit message: collision free border for obstacles

File: aerialist/resources/simulation/box.xacro (robot description, xacro)
@@ -12,7 +12,6 @@
     <collision>
       <geometry>
-        <box size="$(arg l) $(arg w) $(arg h)"/>
+        <box size="${0.8*$(arg l)} ${0.8*$(arg w)} $(arg h)"/>
       </geometry>
-      <!-- <origin xyz="${-$(arg l)/2} ${-$(arg w)/2} ${$(arg h)/2}"/> -->
     </collision>
     <visual>
@@ -20,5 +19,4 @@
         <box size="$(arg l) $(arg w) $(arg h)"/>
       </geometry>
-      <!-- <origin xyz="${-$(arg l)/2} ${-$(arg w)/2} ${$(arg h)/2}"/> -->
     </visual>
     <inertial>
